File: hardware/kicad/bisque-controller.kicad_sch (KiCad schematic)
At the start: 80 parts, among them J1 USB-C, J10 AUX, J2 5V_IN, J3 TC1_K, J4 SSR1, J5 DISPLAY, J6 NAV_SW, J7 AUX, J8 TC2_K, J9 SSR2, Q2 AO3400A, SW1 RESET, SW2 BOOT, U1 ESP32-S3-WROOM-1U-N16R2, U2 AMS1117-3.3, U3 MAX31856MUD+, U4 USBLC6-2SC6, U5 MAX31856MUD+, U6 ULN2003A, U8 LTV-817S-TA1-C, U9 LTV-817S-TA1-C

Commit message: feat(hw): three protected dry-contact inputs with TVS
Generalises rev A's single lid-switch conditioning (R12/R13/C12) into
three identical channels on J11 (lid/gas-flow interlock/spare), each
1k series + 10k pull-up + 100nF, plus one SRV05-4 TVS array (D5)
covering all three raw inputs. Lid moves off J7 onto its own screw
terminal; J7 pin 6 is now unconnected pending Task 11's I2C re-point.

R23-R25 were already taken by Task 8's ULN2003 pulldowns, so the new
resistors use R26-R29 instead of the brief's R23-R26 to avoid silently
overwriting those components. No TVS added to the thermocouple inputs
(Task 6) - array leakage would corrupt the uV-level signal.

Also fixes gen_pcb.py's ROUTE_ORDER, which referenced the now-retired
LID_IN/LID_SW nets and would otherwise KeyError.
Parts:
- added C23, C24: 100nF, Capacitor_SMD:C_0805_2012Metric, symbol Device:C
- added D5: SRV05-4, Package_TO_SOT_SMD:SOT-23-6, symbol Power_Protection:SRV05-4
- added J11: INPUTS, TerminalBlock_Phoenix:TerminalBlock_Phoenix_MKDS-1,5-4-5.08_1x04_P5.08mm_Horizontal, symbol Connector:Screw_Terminal_01x04
- added R26, R28: 1k, Resistor_SMD:R_0805_2012Metric, symbol Device:R
- added R27, R29: 10k, Resistor_SMD:R_0805_2012Metric, symbol Device:R
Connections:
- net LID_SW is gone; now on net IN1: C12.1, R12.2, R13.2
- net +3V3: now also D5.5 (VP), R27.1, R29.1
- net GND: now also C23.2, C24.2, D5.2 (VN), J11.4 (Pin_4)
- net IN2: now also C23.1, R26.2, R27.2
- net IN3: now also C24.1, R28.2, R29.2
- net LID_IN: no longer names the net of J7.6 (Pin_6)
- net LID_IN: no longer R12.1
- new net IN1_RAW: D5.1 (IO1), J11.1 (Pin_1), R12.1
- new net IN2_RAW: D5.3 (IO2), J11.2 (Pin_2), R26.1
- new net IN3_RAW: D5.4 (IO3), J11.3 (Pin_3), R28.1
- no-connect marks 19 -> 21
Other:
- note added: "PROTECTED INPUTS x3 lid/gas-flow/spare (1k + 10k pull-up + 100nF each, SRV05-4 TVS)"
- note removed: "LID SWITCH INPUT FILTER (1k series + 10k pull-up + 100nF)"

Commit message: feat(hw): ADE7953 CT current sensing on I2C
Two current channels, one per SSR zone. Voltage channel unpopulated on a
DNP SELV header so no mains touches the board; true power stays a
firmware-only upgrade later.

Designators corrected against the live COMPONENTS dict (brief's R27-R33/D8
collide with Tasks 7/9): U7, Y1, R30-R38, C25-C37, D6, J12, J13. Interface
strapping, decoupling values, and the QFN-28/crystal footprints follow
hardware/kicad/datasheets/REV-B-NOTES.md's ADE7953 sections, which override
the brief's guessed values throughout - including catching that the brief
had SCLK(25)/~CS(28) swapped onto the real I2C bus pins (26/27 are the
actual SDA/SCL). Crystal load caps (30pF) are an explicitly-flagged
assumption, not a verified datasheet value - see design.py comment.
Parts:
- added C25, C26: 30pF, Capacitor_SMD:C_0805_2012Metric, symbol Device:C
- added C27, C29, C33: 4.7uF, Capacitor_SMD:C_0805_2012Metric, symbol Device:C
- added C28, C30, C34, C36: 100nF, Capacitor_SMD:C_0805_2012Metric, symbol Device:C
- added C31, C32: 33nF, Capacitor_SMD:C_0805_2012Metric, symbol Device:C
- added C35: 10uF, Capacitor_SMD:C_0805_2012Metric, symbol Device:C
- added C37: 1uF, Capacitor_SMD:C_0805_2012Metric, symbol Device:C
- added D6: SRV05-4, Package_TO_SOT_SMD:SOT-23-6, symbol Power_Protection:SRV05-4
- added J12: CT, TerminalBlock_Phoenix:TerminalBlock_Phoenix_MKDS-1,5-4-5.08_1x04_P5.08mm_Horizontal, symbol Connector:Screw_Terminal_01x04
- added J13: AC_SENSE_DNP, Connector_PinHeader_2.54mm:PinHeader_1x02_P2.54mm_Vertical, symbol Connector_Generic:Conn_01x02
- added R30, R37, R38: 10k, Resistor_SMD:R_0805_2012Metric, symbol Device:R
- added R31, R34: 6R8, Resistor_SMD:R_0805_2012Metric, symbol Device:R
- added R32, R33, R35, R36: 1k, Resistor_SMD:R_0805_2012Metric, symbol Device:R
- added U7: ADE7953ACPZ, Package_DFN_QFN:QFN-28-1EP_5x5mm_P0.5mm_EP3.1x3.1mm, symbol Sensor:ADE7953xCP
- added Y1: 3.579545MHz, Crystal:Crystal_SMD_HC49-SD_HandSoldering, symbol Device:Crystal
Connections:
- net +3V3: now also C35.1, C36.1, D6.5 (VP), R30.1, R37.1, R38.1, U7.17 (VDD), U7.7 (PULL_HIGH), U7.8 (PULL_HIGH)
- net I2C_SCL: now also U7.27 (MOSI/SCL/RX)
- net I2C_SDA: now also U7.26 (MISO/SDA/TX)
- net GND renamed ADE_RESET
- net ADE_RESET: now also C25.2, C26.2, C27.2, C28.2, C29.2, C30.2, C31.2, C32.2, C33.2, C34.2, C35.2, C36.2, C37.1, C37.2, D6.2 (VN), R30.2, R33.2, R36.2, U7.10 (IBN), U7.14 (PULL_LOW), U7.16 (AGND), U7.2 (~{RESET}), U7.29 (EP), U7.4 (DGND), U7.6 (IAN)
- new net ADE_CLKIN: C25.1, U7.18 (CLKIN), Y1.1
- new net ADE_CLKOUT: C26.1, U7.19 (CLKOUT), Y1.2
- new net ADE_CS: R38.2, U7.28 (~{CS})
- new net ADE_REF: C33.1, C34.1, U7.13 (REF)
- new net ADE_SCLK: R37.2, U7.25 (SCLK)
- new net ADE_VINTA: C27.1, C28.1, U7.15 (VINTA)
- new net ADE_VINTD: C29.1, C30.1, U7.3 (VINTD)
- new net ADE_VN: J13.2 (Pin_2), U7.11 (VN)
- new net ADE_VP: J13.1 (Pin_1), U7.12 (VP)
- new net CTA_F: C31.1, R32.2, U7.5 (IAP)
- new net CTA_N: D6.3 (IO2), J12.2 (Pin_2), R31.2, R33.1
- new net CTA_P: D6.1 (IO1), J12.1 (Pin_1), R31.1, R32.1
- new net CTB_F: C32.1, R35.2, U7.9 (IBP)
- new net CTB_N: D6.6 (IO4), J12.4 (Pin_4), R34.2, R36.1
- new net CTB_P: D6.4 (IO3), J12.3 (Pin_3), R34.1, R35.1
- no-connect marks 21 -> 27
Other:
- note added: "CT CURRENT SENSING ADE7953, I2C, current-only (no mains - VP/VN to DNP J13)"
