File: hardware/kicad/bisque-controller.kicad_sch (KiCad schematic)
At the start: 115 parts, among them J1 USB-C, J10 AUX, J11 INPUTS, J12 CT, J13 AC_SENSE_DNP, J2 5V_IN, J3 TC1_K, J4 SSR1, J5 DISPLAY, J6 NAV_SW, J7 AUX, J8 TC2_K, J9 SSR2, Q2 AO3400A, SW1 RESET, SW2 BOOT, U1 ESP32-S3-WROOM-1U-N16R2, U2 AMS1117-3.3, U3 MAX31856MUD+, U4 USBLC6-2SC6, U5 MAX31856MUD+, U6 ULN2003A, U7 ADE7953ACPZ, U8 LTV-817S-TA1-C, U9 LTV-817S-TA1-C, Y1 3.579545MHz

Commit message: feat(hw): 14-pin LCD header for touch, plus I2C expansion
Touch controller (XPT2046) is on the display module; only T_CS and T_IRQ
cost new GPIOs (Task 3). T_CLK/T_DIN/T_DO are the shared SPI2 bus, damped
through R39-R43 now that the bus multi-drops four devices at 40 MHz.

J7 pins 5-8 (VENT/AUX_A/AUX_B - dangling single-pin nets nothing on the
board drove) are re-pointed to I2C_SDA/I2C_SCL/+3V3/GND, retiring AUX_A/
AUX_B and giving the I2C bus a 0.1" tap (J7) alongside the new Qwiic
connector (J14), pulled up by R44/R45.

Used R39-R45/J14 rather than the brief's R34-R40, which Task 10 already
consumed. Added the two new footprint snapshots to generator/fp/ and
updated gen_pcb.py's J5/J7 silkscreen label lists and ROUTE_ORDER.

Co-Authored-By: Claude Opus 5 <noreply@anthropic.com>
Parts:
- added J14: QWIIC, Connector_JST:JST_SH_SM04B-SRSS-TB_1x04-1MP_P1.00mm_Horizontal, symbol Connector_Generic:Conn_01x04
- added R39, R40, R41, R42, R43: 33, Resistor_SMD:R_0805_2012Metric, symbol Device:R
- added R44, R45: 4.7k, Resistor_SMD:R_0805_2012Metric, symbol Device:R
- J5: footprint Connector_Molex:Molex_KK-254_AE-6410-08A_1x08_P2.54mm_Vertical -> Connector_Molex:Molex_KK-254_AE-6410-14A_1x14_P2.54mm_Vertical; symbol Connector_Generic:Conn_01x08 -> Connector_Generic:Conn_01x14
Connections:
- net AUX_A is gone; now on net +3V3: J7.7 (Pin_7)
- net AUX_B is gone; now on net ADE_RESET: J7.8 (Pin_8)
- net VENT is gone; now on net I2C_SDA: J7.5 (Pin_5)
- net +3V3: now also J14.2 (Pin_2), R44.1, R45.1
- net ADE_RESET: now also J14.1 (Pin_1)
- net I2C_SCL: now also J7.6 (Pin_6), J14.4 (Pin_4), R45.2
- net I2C_SDA: now also J14.3 (Pin_3), R44.2
- net SPI_MISO: now also J5.9 (Pin_9), R42.1
- net SPI_MOSI: now also R41.1
- net SPI_SCLK: now also R39.1
- net T_CS: now also R40.1
- net T_IRQ: now also R43.1
- new net T_CLK_R: J5.10 (Pin_10), R39.2
- new net T_CS_R: J5.11 (Pin_11), R40.2
- new net T_DIN_R: J5.12 (Pin_12), R41.2
- new net T_DO_R: J5.13 (Pin_13), R42.2
- new net T_IRQ_R: J5.14 (Pin_14), R43.2
- no-connect marks 27 -> 26
Other:
- note added: "HEADERS DISPLAY+TOUCH(J5, 14-pin) NAV(J6) AUX+I2C(J7)"
- note added: "TOUCH DAMPING + I2C EXPANSION (Task 11) R39-43 damp the shared SPI2\nbus for the display module's XPT2046 (not on this board); J14 Qwiic +\nJ7 5-8 (0.1") share the I2C bus, pulled up by R44/R45"
- note removed: "HEADERS DISPLAY(J5) NAV(J6) AUX(J7)"
