File: hardware/kicad/bisque-controller.kicad_sch (KiCad schematic)
At the start: 169 parts, among them J1 USB-C, J10 AUX, J11 INPUTS, J12 CT, J13 AC_SENSE_DNP, J14 QWIIC, J2 24V_IN, J3 TC1_K, J4 SSR1, J5 DISPLAY, J6 NAV_SW, J7 AUX, J8 TC2_K, J9 SSR2, Q2 AO3400A, Q3 AO3400A, Q4 AO3401A, Q5 AO3400A, Q6 AO3400A, SW1 RESET, SW2 BOOT, U1 ESP32-S3-WROOM-1U-N16R2, U10 SN74LVC1G123, U11 XL1509-5.0E1, U2 TLV1117LV33, U3 MAX31856MUD+, U4 SRV05-4, U5 MAX31856MUD+, U6 ULN2003A, U7 ADE7953ACPZ, Y1 3.579545MHz XO

Commit message: hardware: 24 V SSR outputs, opto-driven gates, watchdog in the return
The SSR terminals were "+5 V, watchdog-gated, switched low side" with the
GPIO on the channel MOSFET's gate through 100R - the last place the old
5 V input voltage survived after U11 made the board 24 V. They are now
"24 V, always live, switched low side", the gate is driven through an
optocoupler, and the watchdog sits in the shared return instead of the
supply. 0 DRC violations, 0 unconnected pads, 0 unrouted nets, silk clean
in all four categories, all 14 checkers pass, 12/12 host tests pass.

Three decisions, three derivations - all written up in design.py's SSR
block, which is where the next person will look before re-proposing any
of this.

WHY 24 V. The high side is VIN_P, not VIN: a terminal fed from raw VIN
bypasses the reverse-polarity diode and the fuse, and a screw terminal is
exactly where a wiring mistake lands. F1 holds at 750 mA and U11 takes
~250 mA, so the two channels share ~400 mA; two SSR inputs plus their
indicators is 40 mA, a 10x margin. That budget is a real limit and D9/D10
are sized to it and no further.

WHY THE OPTOCOUPLERS ARE BACK. Not as isolation. The rev B opto-isolation
reversal (93a31d7) is still correct and is not overturned: these terminals
are still board-powered, both sides still share GND, and the pour keepout,
router keepout and check_isolation.py stay gone. What changed is the
failure they are bought for. At 5 V a channel MOSFET failing gate-to-drain
put 5 V through 100R into a GPIO and the clamp survived it; at 24 V the
same single failure puts 240 mA into that clamp and takes the module with
it. The opto removes the conductor - the only thing the MCU touches is an
LED. It is also not more parts than the alternative: a gate-to-GND zener
contains the same fault for the same one part per channel, but by
CONDUCTING, so it has to survive the fault to work and fails open
silently.

The collector sits on SSR_EN (5 V), not on 24 V, and that is load-bearing:
an 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
Parts:
- added D10, D9: 1N4148W, Diode_SMD:D_SOD-123, symbol Device:D
- added Q7: CJ2310, Package_TO_SOT_SMD:SOT-23, symbol Transistor_FET:2N7002
- added R18: 10k, Resistor_SMD:R_0805_2012Metric, symbol Device:R
- added R22: 100k, Resistor_SMD:R_0805_2012Metric, symbol Device:R
- added U8, U9: TLP291, Package_SO:SOP-4_4.4x2.6mm_P1.27mm, symbol Isolator:TLP291
- Q5, Q6: value AO3400A -> CJ2310; symbol Transistor_FET:AO3400A -> Transistor_FET:2N7002; LCSC C20917 -> C75882; MPN C20917 -> C75882
- R10, R21: value 680R -> 4.7k; LCSC C17798 -> C17673; MPN C17798 -> C17673
- R19, R6: value 100R -> 220R; LCSC C17408 -> C17557; MPN C17408 -> C17557
Connections:
- net GND: now also Q7.2 (S), R18.2, R22.2, U8.2, U9.2; no longer Q5.2 (S), Q6.2 (S)
- net SSR1_GATE: now also U8.3; no longer R6.2
- net SSR1_OUT: now also D9.2 (A)
- net SSR2_GATE: now also U9.3; no longer R19.2
- net SSR2_OUT: now also D10.2 (A)
- net SSR_EN: now also Q7.1 (G), R18.1, U8.4, U9.4; no longer J4.1 (Pin_1), J9.1 (Pin_1), LED3.2 (A), LED4.2 (A)
- net VIN_P: now also J4.1 (Pin_1), J9.1 (Pin_1), LED3.2 (A), LED4.2 (A), D10.1 (K), D9.1 (K)
- new net SSR1_LED_A: R6.2, U8.1
- new net SSR2_LED_A: R19.2, U9.1
- new net SSR_RTN: Q5.2 (S), Q6.2 (S), Q7.3 (D), R22.1
Other:
- note added: "HARDWARE WATCHDOG U10 retriggerable one-shot: every rising edge on WDT_KICK restarts a ~2.2 s window, so Q stays high only while firmware keeps kicking. Q holds Q3 on; Q3 pulls SSR_PG down, turning on high-side Q4, which supplies SSR_EN - the +5V GATE DRIVE rail feeding both opto collectors and Q7's gate. R46/C38 set the window. R48 holds B low when the MCU is high-Z. R47 is the fail-safe pull-up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"
- note added: "SSR DRIVE x2 24 V terminals off VIN_P, switched low side by a 60 V CJ2310. The GPIO drives an opto LED, never the gate: at 24 V a gate-to-drain failure would otherwise put 240 mA into the pin. Opto collectors sit on SSR_EN (5 V), so the gate lands at ~4.9 V from the RAIL rather than from CTR. Q7 is the watchdog's gate in the shared return - it opens a channel whose MOSFET failed short. R18/R22 de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"
- note added: "SSR terminals J4/J9: pin1 = VIN_P (24 V, fused and TVS-clamped, ALWAYS LIVE), pin2 = the switched low side. The watchdog gates the shared return (Q7), not the supply, so a tripped watchdog leaves 24 V on pin 1 and opens pin 2. Boot-safe: R7/R20 hold each gate down while the optos are dark. The optos are NOT an isolation barrier - both sides share GND. Rev B's opto-ISOLATED design was reverted and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"
- note removed: "HARDWARE WATCHDOG U10 retriggerable one-shot: every rising edge on WDT_KICK restarts a ~2.2 s window, so Q stays high only while firmware keeps kicking. Q holds Q3 on; Q3 pulls SSR_PG down, turning on high-side Q4, which supplies SSR_EN - the +5V rail feeding BOTH SSR terminals and both indicators. R46/C38 set the window. R48 holds B low when the MCU is high-Z. R47 is the fail-safe pull-up. SJ2 =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"
- note removed: "SSR DRIVE x2 low-side AO3400A; indicator LED across each terminal"
- note removed: "SSR terminals J4/J9: pin1 = SSR_EN (board +5V, watchdog-gated), pin2 = the switched low side. Boot-safe: R7/R20 hold each MOSFET gate down while the ESP32 pins are high-impedance. NOT opto-isolated - rev B tried that and reverted it: an opto only isolates if the SSR loop is powered off-board, and this board powers it. TC1 terminal J3 / TC2 terminal J8: pin1 = K+, pin2 = K- - both float, biased ne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"
- moved on the sheet: BZ1, C12, C18, C19, C20, C21, C22, C23, C24, C25, C27, C28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

Commit message: hardware: the power path loses both its series diodes (Q8, U12)
D1 and D2 were SS34s doing two different jobs, and both had stopped being
the right part for their job.

D1 -> Q8 (AO3401A P-FET) + R62 + D11. VIN_P stopped being a 250 mA net when
the SSR terminals moved to 24 V: it now feeds the buck AND both terminals,
budgeted to 400 mA, so at F1's 750 mA hold the diode burned 0.4 V x 0.65 A
= 260 mW in an SMA. Q8 burns 25 mW at the AO3401A's guaranteed 60 mOhm and
drops ~39 mV, so the SSR block no longer has to excuse a terminal voltage of
"24 V minus a diode". 30 V is enough here where Q5/Q6/Q7 needed 60 V parts,
and the derivation is in design.py: the body diode clamps V_DS forward
before the gate has charged, and D8 clamps a reversed input to ~0.8 V. The
part is Q4's, already Basic, so this adds no feeder fee.

D2 -> U12 (TPS2116) + R63/R64. PRIORITY MODE, not highest-voltage-wins, and
that is the load-bearing part: a 5.25 V host beats a 5.0 V buck, so a plain
ideal diode would hand the relay bank and both SSR terminals to a laptop.
The diode used to prevent that for free by dropping. 30k/10k sets the
switchover at 4.0 V, pinned from both ends - too high and the buck loses its
own priority at the VREF corner, too low and the rail SAGS to the threshold
before USB takes over. U12 also blocks USB back-feeding the unpowered buck,
which closes fab-review finding C1 in design rather than on the bench.

The buck's output becomes its own net, BUCK_5V, so C44/C45/C46 stay on the
regulator's side of the mux where its compensation needs them.

U12 is the first fine-pitch part here whose escapes carry RAILS rather than
signals, and that needed two mechanisms: gen_pcb.FANOUT (without it the pads
report "0 goal node(s), free neighbours F/B=0/0", exactly as U10 did) and
MUX_SEEDS/MUX_TERMS, because a 0.7 mm track centred 0.5 mm from a 0.25 mm
stub leaves 0.025 mm where 0.2 mm is needed. Rot 180 rather than 0 so the
two corner pads that carry a net escape north instead of south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
Parts:
- removed D1, D2: SS34, Diode_SMD:D_SMA, symbol Device:D_Schottky
- added D11: BZT52C8V2, Diode_SMD:D_SOD-323, symbol Device:D_Zener
- added Q8: AO3401A, Package_TO_SOT_SMD:SOT-23, symbol Transistor_FET:AO3401A
- added R62: 100k, Resistor_SMD:R_0805_2012Metric, symbol Device:R
- added R63: 30k, Resistor_SMD:R_0805_2012Metric, symbol Device:R
- added R64: 10k, Resistor_SMD:R_0805_2012Metric, symbol Device:R
- added U12: TPS2116DRLR, Package_TO_SOT_SMD:SOT-583-8, symbol Power_Management:TPS2116DRL
Connections:
- net +5V: now also U12.2 (VOUT), U12.7 (VOUT); no longer C44.1, C45.1, C46.1, L1.1, U11.3 (FB)
- net GND: now also R62.2, R64.2, U12.1 (GND)
- net VBUS: now also U12.6 (VIN2)
- net VIN_F: now also Q8.3 (D)
- net VIN_P: now also D11.1 (K), Q8.2 (S)
- new net BUCK_5V: C44.1, C45.1, C46.1, L1.1, R63.1, U11.3 (FB), U12.3 (VIN1), U12.5 (MODE)
- new net MUX_PR1: R63.2, R64.1, U12.4 (PR1)
- new net VIN_GATE: D11.2 (A), Q8.1 (G), R62.1
- no-connect marks 28 -> 29
Other:
- note added: "POWER IN 24 VDC terminal or USB F1+D8 clamp-and-blow at the entry. Q8 blocks reverse polarity as a P-FET, not a diode: its body diode conducts on correct polarity and the gate then pulls itself on through R62, clamped by D11 because 24 V is twice the AO3401A's V_GS rating. U11 (right) makes BUCK_5V; U12 selects between it and USB VBUS to make +5V, giving the buck PRIORITY via R63/R64 rather than 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"
- note removed: "POWER IN 24 VDC terminal or USB F1+D8 clamp-and-blow at the entry; D1 blocks reverse polarity. U11 (right) makes +5V; D2 ORs in USB VBUS; U2 drops it to +3V3"
- moved on the sheet: BZ1, C1, C10, C11, C12, C13, C14, C15, C16, C17, C18, C19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

Commit message: hardware: regenerate the schematic for C47/C48 and the SSR resistor values
gen_sch.py output for design.py at 7b98b98. The board, fab outputs and
renders follow once the full route and every checker pass.

Co-Authored-By: Claude Opus 5.5 <noreply@anthropic.com>
Claude-Session: https://claude.ai/code/session_01UdnA6LQkwHR1vk19fXPp5i
Parts:
- added C47, C48: 1uF, Capacitor_SMD:C_0402_1005Metric, symbol Device:C
- R10, R21: value 4.7k -> 10k; LCSC C17673 -> C17414; MPN C17673 -> C17414
- R20, R7: value 10k -> 4.7k; LCSC C17414 -> C17673; MPN C17414 -> C17673
Connections:
- net BUCK_5V: now also C48.1
- net GND: now also C47.2, C48.2
- net VBUS: now also C47.1
Other:
- moved on the sheet: C1, C11, C2, C3, C4, C41, C42, C43, C44, C45, C46, C5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

Commit message: hardware: the schematic becomes hierarchical, one sheet per functional area
gen_sch.py's last run: a root sheet indexing seven A3/A2 sub-sheets
(power, mcu, thermocouples, ssr, io, ct, test) built from the existing
GROUPS taxonomy. Nets cross sheets as the global labels they already
were; rails stay power ports; block-local nets stay fused wires with
local labels. Power flags now live beside the net they flag - on one
flat sheet a flag's global label merged with the block's local label by
name, across sheets it would not. #PWR numbering runs across sheets so
KiCad sees no annotation error, and a block taller than its column is
an overflow (the CT sheet lands on A2) rather than a clipped page.

The exported netlist is identical to design.py's on every net, footprint
and value; ERC reports exactly the flat sheet's four pre-existing items.
check_sch_bounds / check_sch_layout / check_sch_uuids / check_mpn now walk
every sheet reachable from the root.

Co-Authored-By: Claude Fable 5.1 <noreply@anthropic.com>
Parts:
- removed BZ1: active 5V, Buzzer_Beeper:Buzzer_12x9.5RM7.6, symbol Device:Buzzer
- removed C1, C3: 22uF/25V, Capacitor_SMD:C_1206_3216Metric, symbol Device:C
- removed C10, C12, C13, C14, C15, C18, C19, C2, C20, C23, C24, C25, C28, C30, C34, C36, C39, C4, C43, C6: 100nF, Capacitor_SMD:C_0805_2012Metric, symbol Device:C
- removed C11, C35, C7: 10uF, Capacitor_SMD:C_0805_2012Metric, symbol Device:C
- removed C16, C17, C21, C22: 10nF, Capacitor_SMD:C_0805_2012Metric, symbol Device:C
- removed C27, C29, C33: 4.7uF, Capacitor_SMD:C_0805_2012Metric, symbol Device:C
- removed C31, C32, C40: 33nF, Capacitor_SMD:C_0805_2012Metric, symbol Device:C
- removed C37, C5: 1uF, Capacitor_SMD:C_0805_2012Metric, symbol Device:C
- removed C38, C44, C45: 22uF, Capacitor_SMD:C_1206_3216Metric, symbol Device:C
- removed C41, C42: 10uF/50V, Capacitor_SMD:C_1206_3216Metric, symbol Device:C
- removed C46: 100uF/16V, Capacitor_SMD:CP_Elec_5x5.4, symbol Device:C_Polarized
- removed C47, C48: 1uF, Capacitor_SMD:C_0402_1005Metric, symbol Device:C
- removed D10, D3, D4, D9: 1N4148W, Diode_SMD:D_SOD-123, symbol Device:D
- removed D11: BZT52C8V2, Diode_SMD:D_SOD-323, symbol Device:D_Zener
- removed D5, D6, U4: SRV05-4, Package_TO_SOT_SMD:SOT-23-6, symbol Power_Protection:SRV05-4
- removed D7: SS34, Diode_SMD:D_SMA, symbol Device:D_Schottky
- removed D8: SMAJ30A, Diode_SMD:D_SMA, symbol Device:D_TVS
- removed F1: 750mA/33V, Fuse:Fuse_1812_4532Metric, symbol Device:Polyfuse
- removed FID1, FID2, FID3: FIDUCIAL, Fiducial:Fiducial_1mm_Mask2mm, symbol Mechanical:Fiducial
- removed H1, H2, H3, H4: M3, MountingHole:MountingHole_3.2mm_M3_Pad_Via, symbol Mechanical:MountingHole_Pad
- removed J1: USB-C, Connector_USB:USB_C_Receptacle_HRO_TYPE-C-31-M-12, symbol Connector:USB_C_Receptacle_USB2.0_16P
- removed J10: AUX, TerminalBlock_Phoenix:TerminalBlock_Phoenix_MKDS-1,5-4-5.08_1x04_P5.08mm_Horizontal, symbol Connector:Screw_Terminal_01x04
- removed J11: INPUTS, TerminalBlock_Phoenix:TerminalBlock_Phoenix_MKDS-1,5-4-5.08_1x04_P5.08mm_Horizontal, symbol Connector:Screw_Terminal_01x04
- removed J12: CT, TerminalBlock_Phoenix:TerminalBlock_Phoenix_MKDS-1,5-4-5.08_1x04_P5.08mm_Horizontal, symbol Connector:Screw_Terminal_01x04
- removed J13: AC_SENSE_DNP, Connector_PinHeader_2.54mm:PinHeader_1x02_P2.54mm_Vertical, symbol Connector_Generic:Conn_01x02
- removed J14: QWIIC, Connector_JST:JST_SH_SM04B-SRSS-TB_1x04-1MP_P1.00mm_Horizontal, symbol Connector_Generic_MountingPin:Conn_01x04_MountingPin
- removed J2: 24V_IN, TerminalBlock_Phoenix:TerminalBlock_Phoenix_MKDS-1,5-2-5.08_1x02_P5.08mm_Horizontal, symbol Connector:Screw_Terminal_01x02
- removed J3: TC1_K, TerminalBlock_Phoenix:TerminalBlock_Phoenix_MKDS-1,5-2-5.08_1x02_P5.08mm_Horizontal, symbol Connector:Screw_Terminal_01x02
- removed J4: SSR1, TerminalBlock_Phoenix:TerminalBlock_Phoenix_MKDS-1,5-2-5.08_1x02_P5.08mm_Horizontal, symbol Connector:Screw_Terminal_01x02
- removed J5: DISPLAY, Connector_Molex:Molex_KK-254_AE-6410-14A_1x14_P2.54mm_Vertical, symbol Connector_Generic:Conn_01x14
- removed J6: NAV_SW, Connector_Molex:Molex_KK-254_AE-6410-06A_1x06_P2.54mm_Vertical, symbol Connector_Generic:Conn_01x06
- removed J7: AUX, Connector_Molex:Molex_KK-254_AE-6410-08A_1x08_P2.54mm_Vertical, symbol Connector_Generic:Conn_01x08
- removed J8: TC2_K, TerminalBlock_Phoenix:TerminalBlock_Phoenix_MKDS-1,5-2-5.08_1x02_P5.08mm_Horizontal, symbol Connector:Screw_Terminal_01x02
- removed J9: SSR2, TerminalBlock_Phoenix:TerminalBlock_Phoenix_MKDS-1,5-2-5.08_1x02_P5.08mm_Horizontal, symbol Connector:Screw_Terminal_01x02
- removed L1: 47uH/2A, Inductor_SMD:L_Changjiang_FXL0650, symbol Device:L
- removed LED1: WS2812B, LED_SMD:LED_WS2812B_PLCC4_5.0x5.0mm_P3.2mm, symbol LED:WS2812B
- removed LED2: green, LED_SMD:LED_0805_2012Metric, symbol Device:LED
- removed LED3, LED4: amber, LED_SMD:LED_0805_2012Metric, symbol Device:LED
- removed Q2, Q3: AO3400A, Package_TO_SOT_SMD:SOT-23, symbol Transistor_FET:AO3400A
- removed Q4, Q8: AO3401A, Package_TO_SOT_SMD:SOT-23, symbol Transistor_FET:AO3401A
- removed Q5, Q6, Q7: CJ2310, Package_TO_SOT_SMD:SOT-23, symbol Transistor_FET:2N7002
- removed R1, R10, R13, R18, R2, R21, R23, R24, R25, R27, R29, R30, R37, R38, R50, R51, R52, R53, R64, R8: 10k, Resistor_SMD:R_0805_2012Metric, symbol Device:R
- removed R11: 100R, Resistor_SMD:R_0805_2012Metric, symbol Device:R
- removed R12, R26, R28, R32, R33, R35, R36, R59, R60, R61, R9: 1k, Resistor_SMD:R_0805_2012Metric, symbol Device:R
- removed R14, R15, R16, R17: 100R 1%, Resistor_SMD:R_0805_2012Metric, symbol Device:R
- removed R19, R6: 220R, Resistor_SMD:R_0805_2012Metric, symbol Device:R
- removed R20, R44, R45, R7: 4.7k, Resistor_SMD:R_0805_2012Metric, symbol Device:R
- removed R22, R46, R47, R48, R49, R62: 100k, Resistor_SMD:R_0805_2012Metric, symbol Device:R
- removed R3: 330R, Resistor_SMD:R_0805_2012Metric, symbol Device:R
- removed R31, R34: 5R1, Resistor_SMD:R_0805_2012Metric, symbol Device:R
- removed R39, R40, R41, R42, R43, R54, R55, R56, R57, R58: 33, Resistor_SMD:R_0805_2012Metric, symbol Device:R
- removed R4, R5: 5.1k, Resistor_SMD:R_0805_2012Metric, symbol Device:R
- removed R63: 30k, Resistor_SMD:R_0805_2012Metric, symbol Device:R
- removed SJ1: AUX_VP=5V, Jumper:SolderJumper-2_P1.3mm_Open_RoundedPad1.0x1.5mm, symbol Jumper:SolderJumper_2_Open
- removed SJ2: WDT_DEFEAT, Jumper:SolderJumper-2_P1.3mm_Open_RoundedPad1.0x1.5mm, symbol Jumper:SolderJumper_2_Open
- removed SW1: RESET, Button_Switch_SMD:SW_Push_1P1T_XKB_TS-1187A, symbol Switch:SW_Push
- removed SW2: BOOT, Button_Switch_SMD:SW_Push_1P1T_XKB_TS-1187A, symbol Switch:SW_Push
- removed TP1, TP10, TP11, TP12, TP2, TP3, TP4, TP5, TP6, TP7, TP8, TP9: TP, TestPoint:TestPoint_Pad_D1.0mm, symbol Connector:TestPoint
- removed U1: ESP32-S3-WROOM-1U-N16R2, RF_Module:ESP32-S3-WROOM-1U, symbol RF_Module:ESP32-S3-WROOM-1
- removed U10: SN74LVC1G123, Package_SO:SSOP-8_2.95x2.8mm_P0.65mm, symbol 74xGxx:74LVC1G123
- removed U11: XL1509-5.0E1, Package_SO:SOIC-8_3.9x4.9mm_P1.27mm, symbol Regulator_Switching:XL1509-5.0
- removed U12: TPS2116DRLR, Package_TO_SOT_SMD:SOT-583-8, symbol Power_Management:TPS2116DRL
- removed U2: TLV1117LV33, Package_TO_SOT_SMD:SOT-223-3_TabPin2, symbol Regulator_Linear:TLV1117-33
- removed U3, U5: MAX31856MUD+, Package_SO:TSSOP-14_4.4x5mm_P0.65mm, symbol Sensor_Temperature:MAX31856
- removed U6: ULN2003A, Package_SO:SOIC-16_3.9x9.9mm_P1.27mm, symbol Transistor_Array:ULN2003A
- removed U7: ADE7953ACPZ, Package_DFN_QFN:QFN-28-1EP_5x5mm_P0.5mm_EP3.1x3.1mm, symbol Sensor:ADE7953xCP
- removed U8, U9: TLP291, Package_SO:SOP-4_4.4x2.6mm_P1.27mm, symbol Isolator:TLP291
- removed Y1: 3.579545MHz XO, Oscillator:Oscillator_SMD_Abracon_ASE-4Pin_3.2x2.5mm, symbol Oscillator:ASE-xxxMHz
Connections:
- no-connect marks 29 -> 0
Other:
- added sheet ct (sheets/ct.kicad_sch)
- added sheet io (sheets/io.kicad_sch)
- added sheet mcu (sheets/mcu.kicad_sch)
- added sheet power (sheets/power.kicad_sch)
- added sheet ssr (sheets/ssr.kicad_sch)
- added sheet test (sheets/test.kicad_sch)
- added sheet thermocouples (sheets/thermocouples.kicad_sch)
- note removed: "24 V -> 5 V BUCK XL1509-5.0, fixed output C41-C43 in, D7 catch, L1 47uH, C44/C45/C46 out. FB ties to the output because the part is the fixed 5.0 V version; EN is active LOW and grounded. C46 is an ELECTROLYTIC on purpose: voltage-mode with fixed compensation needs its ESR zero, and an all-ceramic output has none. Keep C41/C42 - U11 - D7 tight: that loop, not L1, is what radiates."
- note removed: "ALARM BUZZER"
- note removed: "AUX OUTPUT BANK ULN2003 vent/purge/spare; COM->AUX_VP, SJ1 links to +5V"
- note removed: "CT CURRENT SENSING ADE7953, I2C, current-only no mains - VP/VN to DNP J13"
- note removed: "ESP32-S3-WROOM-1U-N16R2 GPIOs = firmware Kconfig defaults"
- note removed: "HARDWARE WATCHDOG U10 retriggerable one-shot: every rising edge on WDT_KICK restarts a ~2.2 s window, so Q stays high only while firmware keeps kicking. Q holds Q3 on; Q3 pulls SSR_PG down, turning on high-side Q4, which supplies SSR_EN - the +5V GATE DRIVE rail feeding both opto collectors and Q7's gate. R46/C38 set the window. R48 holds B low when the MCU is high-Z. R47 is the fail-safe pull-up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"
- note removed: "HEADERS J5 display+touch (14-pin), J6 nav, J7 aux+I2C"
- note removed: "MOUNTING / FIDUCIALS / POWER FLAGS FID1-3 are bare-copper pick-and-place targets, on no net"
- note removed: "POWER IN 24 VDC terminal or USB F1+D8 clamp-and-blow at the entry. Q8 blocks reverse polarity as a P-FET, not a diode: its body diode conducts on correct polarity and the gate then pulls itself on through R62, clamped by D11 because 24 V is twice the AO3401A's V_GS rating. U11 (right) makes BUCK_5V; U12 selects between it and USB VBUS to make +5V, giving the buck PRIORITY via R63/R64 rather than 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"
- note removed: "PROTECTED INPUTS x3 lid / gas-flow / spare 1k + 10k pull-up + 100nF each, SRV05-4 TVS"
- note removed: "RESET / BOOT / DECOUPLING"
- note removed: "SPI BUS DAMPING + CHIP-SELECT PULL-UPS + I2C EXPANSION R39-R43 damp the display module's XPT2046 touch lines and R54-R58 the four 40 MHz display lines; both loom to J5. R56 is also the SDO hedge - lift it if the panel does not tri-state J5.9 off the shared SPI_MISO. R50-R53 hold all four chip selects deasserted from power-on, before firmware configures any GPIO. J14 Qwiic and J7 5-8 (0.1 in) shar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"
- note removed: "SSR DRIVE x2 24 V terminals off VIN_P, switched low side by a 60 V CJ2310. The GPIO drives an opto LED, never the gate: at 24 V a gate-to-drain failure would otherwise put 240 mA into the pin. Opto collectors sit on SSR_EN (5 V), so the gate lands at ~4.9 V from the RAIL rather than from CTR. Q7 is the watchdog's gate in the shared return - it opens a channel whose MOSFET failed short. R18/R22 de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"
- note removed: "TEST POINTS"
- note removed: "THERMOCOUPLE 1 (control) MAX31856 T- floats to J3, biased via BIAS"
- note removed: "THERMOCOUPLE 2 (load) MAX31856 T- floats to J8, biased via BIAS"
- note removed: "USB-C native USB flashing + ESD"
- note removed: "WS2812B STATUS LED VDD dropped ~4.6V for 3.3V data margin"
