File: hardware/kicad/sheets/ct.kicad_sch (KiCad schematic)
At the start: 30 parts, among them J12 CT, U7 ADE7953ACPZ, Y1 3.579545MHz XO

Commit message: hardware: BOM from the schematic, JLCPCB fits every part
BOM.csv is now kicad-cli's export of the schematic itself (make pcb-fab),
so every symbol not marked "Exclude from BOM" is on it; gen_jlc reads the
same flags instead of a hand-kept NOT_ASSEMBLED/HAND_SOLDER table.

JLCPCB assembly of the 12 through-hole parts plus LED1 costs ~$22 an order
against ~$110 for partial assembly and a Mouser order, so they are no
longer hand-fitted. Their Assembly field reads "Optional hand solder - JLC
assembles; untick at JLC to fit by hand"; setting it back to "HAND SOLDER"
makes a part hand-fitted again. JLC_PLACEMENT gains fitted corrections for
the six new LCSC parts (J7 needs 180 deg).

LED1 moves to the in-stock WS2812B-V5/W (C2874885): same pinout, and its
VIH of 0.63*VDD (~2.6 V at VLED) is below the old part's 2.7 V.
mouser-order.csv now holds only the mating housings and crimps.

Co-Authored-By: Claude Opus 5.5 <noreply@anthropic.com>
Parts:
- J12: Assembly (none) -> Optional hand solder - JLC assembles; untick at JLC to fit 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
Changed lines of the file:
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@@
 			)
 		)
-	)
+		(property "Assembly" "Optional hand solder - JLC assembles; untick at JLC to fit by hand"
+			(at 15.24 190.5 0)
+			(hide yes)
+			(effects
+				(font
+					(size 1.27 1.27)
+				)
+			)
+		))
 	(symbol
 		(lib_id "Device:C")
