File: hardware/kicad/sheets/mcu.kicad_sch (KiCad schematic)
At the start: 42 parts, among them J1 USB-C, J14 QWIIC, J5 DISPLAY, J6 NAV_SW, J7 AUX, SW1 RESET, SW2 BOOT, U1 ESP32-S3-WROOM-1U-N16R2, U4 SRV05-4

Commit message: hardware: SPI return paths - source series R72/R73, transfer caps C51-C54, GND stitching (PCB review 2026-10-05 item 5)
The stack puts F.Cu over the GND plane and B.Cu over the +3V3 plane, so
every one of the bus's 34 layer transitions was a reference change with
the nearest 3V3-GND capacitor 10-46 mm away and no GND via beside it.

Re-routing was tried first, eight ways on scratch copies (via cost
12-160, every net order, with and without the chip selects and LCD lines
ripped): the corridor between U1 and the J5 rows forces 7-13 vias per
net whatever the penalty, and the runs that cut vias doubled the length.
The committed routing stays; the review's other three levers are applied:

- R72/R73 (33R 0603, C23140, Basic) between U1's SCLK/MOSI pins and the
  bus, ahead of every branch. The SCLK junction was on the pad itself,
  so its east run to U3/U5 is re-grown from behind the resistor (11 -> 13
  vias) and MISO's escape moves to clear R72. Pin-side stubs are
  SPI_SCLK_U1 / SPI_MOSI_U1 (locked copper); check_pinmap and
  pin-assignments.md follow. MISO stays bare: its damping is at the slaves.
- C51-C54 (100nF 0603 X7R, C14663, Basic), each with its own via to each
  plane, at the four sites a cap plus two vias fits within 3 mm of a bus
  via: 5 of 37 bus vias within 3 mm of a transfer cap (was 0 of 34),
  farthest bus via from any 3V3-GND cap 36 mm (was 46). The U1 exit
  cluster and the J5 rows have no room; said so in the notes.
- 29 GND stitch vias: 26 of 42 SPI+T_CS vias now have one within 1.5 mm
  (was 1 of 39). A GND via bridges In1 to the outer pours, not to +3V3,
  and the notes say what that does and does not buy.
- Bench: "SPI bus waveforms at 40 MHz" in bench-smoke-test.md with the
  tuning order (R54/R55 to 0R, then R72/R73 to 47R, then 20 MHz).

Side effects: BOM 50 -> 52 lines (two Basic 0603 lines), nameplate
pocket shrank so the silk nameplate prints at 62 %. Two route.py gaps
found and documented (DESIGN-NOTES "Tooling notes"): a net with two
FA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
Parts:
- added C51, C52, C53, C54: 100nF, Capacitor_SMD:C_0603_1608Metric, symbol Device:C
- added R72, R73: 33, Resistor_SMD:R_0603_1608Metric, symbol Device:R
Connections:
- net +3V3: now also C51.1, C52.1, C53.1, C54.1
- net GND: now also C51.2, C52.2, C53.2, C54.2
- net SPI_MOSI: now also R73.2; no longer U1.19 (IO11)
- net SPI_SCLK: now also R72.2; no longer U1.20 (IO12)
- new net SPI_MOSI_U1: R73.1, U1.19 (IO11)
- new net SPI_SCLK_U1: R72.1, U1.20 (IO12)
Other:
- note added: "SPI BUS DAMPING + CHIP-SELECT PULL-UPS + I2C EXPANSION R39-R43 damp the display module's XPT2046 touch lines and R54-R58 the four 40 MHz display lines; both loom to J5. R72/R73 series-terminate SCLK and MOSI at U1's own pins, ahead of every branch: SPI_SCLK_U1/SPI_MOSI_U1 are the pin-side stubs. R56 is also the SDO hedge - lift it if the panel does not tri-state J5.9 off the shared SPI_MISO. R50-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"
- note added: "SPI RETURN-PATH CAPS (PCB review 2026-10-05 item 5) C51-C54 sit on the board at the SPI bus's F.Cu/B.Cu transitions, not at U1: a signal that changes outer layer changes reference plane (In1 GND to In2 +3V3), and the return current crosses between the planes through the nearest 3V3-GND capacitor. One 0603 per via cluster, each with its own via to each plane."
- note removed: "SPI BUS DAMPING + CHIP-SELECT PULL-UPS + I2C EXPANSION R39-R43 damp the display module's XPT2046 touch lines and R54-R58 the four 40 MHz display lines; both loom to J5. R56 is also the SDO hedge - lift it if the panel does not tri-state J5.9 off the shared SPI_MISO. R50-R53 hold all four chip selects deasserted from power-on, before firmware configures any GPIO. J14 Qwiic and J7 5-8 (0.1 in) shar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"

Commit message: hardware: BOM from the schematic, JLCPCB fits every part
BOM.csv is now kicad-cli's export of the schematic itself (make pcb-fab),
so every symbol not marked "Exclude from BOM" is on it; gen_jlc reads the
same flags instead of a hand-kept NOT_ASSEMBLED/HAND_SOLDER table.

JLCPCB assembly of the 12 through-hole parts plus LED1 costs ~$22 an order
against ~$110 for partial assembly and a Mouser order, so they are no
longer hand-fitted. Their Assembly field reads "Optional hand solder - JLC
assembles; untick at JLC to fit by hand"; setting it back to "HAND SOLDER"
makes a part hand-fitted again. JLC_PLACEMENT gains fitted corrections for
the six new LCSC parts (J7 needs 180 deg).

LED1 moves to the in-stock WS2812B-V5/W (C2874885): same pinout, and its
VIH of 0.63*VDD (~2.6 V at VLED) is below the old part's 2.7 V.
mouser-order.csv now holds only the mating housings and crimps.

Co-Authored-By: Claude Opus 5.5 <noreply@anthropic.com>
Parts:
- J5, J6, J7: Assembly (none) -> Optional hand solder - JLC assembles; untick at JLC to fit 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
- LED1: Assembly (none) -> Optional hand solder - JLC assembles; untick at JLC to fit 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; LCSC C2761795 -> C2874885; MPN WS2812B-B/T -> WS2812B-V5/W
- TP10, TP4, TP5, TP6, TP9: now left out of the parts list
Changed lines of the file:
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@@
 			)
 		)
-	)
+		(property "Assembly" "Optional hand solder - JLC assembles; untick at JLC to fit by hand"
+			(at 378.46 52.07 0)
+			(hide yes)
+			(effects
+				(font
+					(size 1.27 1.27)
+				)
+			)
+		))
 	(symbol
 		(lib_id "power:+3V3")
@@
 		(unit 1)
 		(exclude_from_sim no)
-		(in_bom yes)
+		(in_bom no)
 		(on_board yes)
 		(dnp no)
@@
 		(unit 1)
 		(exclude_from_sim no)
-		(in_bom yes)
+		(in_bom no)
 		(on_board yes)
 		(dnp no)
@@
 		(unit 1)
 		(exclude_from_sim no)
-		(in_bom yes)
+		(in_bom no)
 		(on_board yes)
 		(dnp no)
@@
 		(unit 1)
 		(exclude_from_sim no)
-		(in_bom yes)
+		(in_bom no)
 		(on_board yes)
 		(dnp no)
@@
 			)
 		)
-		(property "Datasheet" "https://datasheet.lcsc.com/datasheet/pdf/bc8264a6d62c958a89e25ec8cc82b690.pdf?productCode=C2761795"
+		(property "Datasheet" "https://datasheet.lcsc.com/datasheet/pdf/3795cfb9d54f7ec8ecc0b043ede3c05a.pdf?productCode=C2874885"
 			(at 163.83 207.01 0)
 			(hide yes)
@@
 			)
 		)
-		(property "MPN" "WS2812B-B/T"
+		(property "MPN" "WS2812B-V5/W"
 			(at 163.83 207.01 0)
 			(hide yes)
@@
 			)
 		)
-		(property "LCSC" "C2761795"
+		(property "LCSC" "C2874885"
 			(at 163.83 207.01 0)
 			(hide yes)
@@
 			)
 		)
-	)
+		(property "Assembly" "Optional hand solder - JLC assembles; untick at JLC to fit by hand"
+			(at 163.83 207.01 0)
+			(hide yes)
+			(effects
+				(font
+					(size 1.27 1.27)
+				)
+			)
+		))
 	(symbol
 		(lib_id "Device:R")
@@
 			)
 		)
-	)
+		(property "Assembly" "Optional hand solder - JLC assembles; untick at JLC to fit by hand"
+			(at 304.8 59.69 0)
+			(hide yes)
+			(effects
+				(font
+					(size 1.27 1.27)
+				)
+			)
+		))
 	(symbol
 		(lib_id "Device:R")
@@
 		(unit 1)
 		(exclude_from_sim no)
-		(in_bom yes)
+		(in_bom no)
 		(on_board yes)
 		(dnp no)
@@
 			)
 		)
-	)
+		(property "Assembly" "Optional hand solder - JLC assembles; untick at JLC to fit by hand"
+			(at 337.82 46.99 0)
+			(hide yes)
+			(effects
+				(font
+					(size 1.27 1.27)
+				)
+			)
+		))
 	(symbol
 		(lib_id "Device:C")
