File: hardware/kicad/sheets/power.kicad_sch (KiCad schematic)
At the start: 30 parts, among them J2 24V_IN, Q8 AO3401A, U11 XL1509-5.0E1, U12 TPS2116DRLR, U2 TLV1117LV33

Commit message: hardware: qualify the 24 V -> 5 V buck (PCB review 2026-10-05 item 3)
Input: C41/C42 are now CL32B475KBUYNNE 1210 X7R 4.7 uF (C170099), chosen
on Samsung's DC-bias curve - 3.10 uF each at 24 V, 2.72 at 29 V - where
the 1206 X5R 10 uF they replace held 1.35 uF. 6.2 uF for the pair, 0.43 A
rms, 0.23 V pp. No input electrolytic, deliberately: a GP can's ripple
share cannot be bounded without a 100 kHz ESR (DESIGN-NOTES at C41).

Output: C46 is the Panasonic FK EEEFK1E101SP (C178540), 100 uF/25 V with
0.36 ohm and 240 mA SPECIFIED at 100 kHz - the LM2596-table class - in
place of a general-purpose RVT whose sheet gave only tan d at 120 Hz.
C45 is removed: one 22 uF ceramic puts the takeover of the ESR zero at
32 kHz instead of 16 kHz. Output-filter phase at 10/20/40 kHz is now
-124/-129/-143 deg against -148/-163/-172 before. The error amplifier
is unpublished, so loop stability is written as a bench item (load step,
startup, no/full load, hot) in docs/bench-smoke-test.md.

Layout: U11 turned 180 so the switch pin faces D7 and L1; SW_5V is 9.4 mm
of F.Cu in two legs with no via (was 18 mm, two layer changes), locked;
C41 2.5 mm from pin 1 with its GND via beside it, D7's anode on two vias,
FB from C44's pad on B.Cu; VIN_P and BUCK_5V cross the block on B.Cu;
FID3 moved 3.9 mm south for the 6.3 mm can.

Budget: the 5 V rail is rated 1.0 A at 50 C ambient. At 29 V, 127 kHz and
L -20% the inductor peak is 1.48 A against the 2.08 A 30%-drop point;
U11 ~0.6 W, D7 0.53 W. The regulator's 2 A headline is not a rating.

ERC 0, DRC 0, unconnected 0, via/pad PASS, sync idempotent, uuid round
trip 0 minted, manifest 29/29 (two sheets added, two retired). 50 BOM
lines, Standard $110.27, unchanged; one more Extended line on Economic.

Co-Authored-By: Claude Fable 5.1 <noreply@anthropic.com>
Parts:
- removed C45: 22uF/25V, Capacitor_SMD:C_1206_3216Metric, symbol Device:C
- C41, C42: value 10uF/50V -> 4.7uF/50V; footprint Capacitor_SMD:C_1206_3216Metric -> Capacitor_SMD:C_1210_3225Metric; LCSC C13585 -> C170099; MPN CL31A106KBHNNNE -> CL32B475KBUYNNE
- C46: value 100uF/16V -> 100uF/25V; footprint Capacitor_SMD:CP_Elec_5x5.4 -> Capacitor_SMD:CP_Elec_6.3x5.8; LCSC C2977550 -> C178540; MPN RVT1C101M0505 -> EEEFK1E101SP; Manufacturer ROQANG -> PANASONIC
Other:
- note added: "24 V -> 5 V BUCK XL1509-5.0, fixed output (LM2596 class) C41/C42 in (1210 X7R: 3.1 uF each AT 24 V - a 1206 10 uF held 1.35), D7 catch, L1 47uH, C44 + C46 out. FB ties to the output because the part is the fixed 5.0 V version; EN is active LOW and grounded. C46 is a LOW-IMPEDANCE ELECTROLYTIC on purpose, 0.36 ohm AT 100 kHz: voltage-mode with fixed compensation leans on its ESR zero (4.4 kHz), an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"
- note removed: "24 V -> 5 V BUCK XL1509-5.0, fixed output C41-C43 in, D7 catch, L1 47uH, C44/C45/C46 out. FB ties to the output because the part is the fixed 5.0 V version; EN is active LOW and grounded. C46 is an ELECTROLYTIC on purpose: voltage-mode with fixed compensation needs its ESR zero, and an all-ceramic output has none. Keep C41/C42 - U11 - D7 tight: that loop, not L1, is what radiates."

Commit message: hardware: VBUS bulk C50, and the USB clamp coordinated honestly (PCB review 2026-10-05 item 6)
The review was right that "U4 clamps transients so U12 is safe" was
unsupported: the SRV05-4's rail clamp breaks down at 6 V minimum and
clamps at 13.5 V at 4 A, so nothing in it holds VBUS under the
TPS2116's 6 V absolute maximum. What does is charge sharing. The
exposure is defined as IEC 61000-4-2 +-8 kV contact at a bench port
inside the enclosure (no 61000-4-5 claim); an 8 kV gun's 1.2 uC lands
on the VBUS node whichever pin it hits, because U4 steers D+/D- there,
and with C47 alone (0.55 uF at 5 V on Samsung's curve) that was a 2.2 V
step - 7.2-7.5 V on a 6 V pin.

C50: 4.7 uF 25 V X5R 0805 (C1779, already the C27/C29/C33 line, Basic;
3.20 uF at 5 V) across VBUS at (52.4, 31.1) under J1, pad 1 on the
locked VBUS trunk, pad 2 on its own GND via. 3.75 uF on the node makes
the step 0.32 V, 5.3-5.6 V peak. Not 10 uF: that part keeps 4.97 uF at
5 V for 0.1 V of gain and puts the port at 11 uF / 55 uC against USB's
10 uF / 50 uC; the land takes it if the bench wants it. The same
capacitance lowers sqrt(L/C) for the hot-plug ring from 1.35 to
0.52 ohm; the smoke test now scopes VBUS at C50 on insertion with the
10 uF swap as the fallback. Said plainly at C50 and U4: a sustained
>6 V from a defective host is not covered (rev C: an OVP load switch).
Hold-up restated (0.5 A x 8 us into ~25 uF = 160 mV); no VOUT cap.

Schematic: C50 on the power sheet with its own VBUS/GND symbols, the
power-in note extended; the Konnect-added symbols were rebuilt from
their neighbours' form (field offsets, pin uuids, instance path) so
ERC, check_sch_layout and the uuid round-trip all pass. Board: DRC 0,
unconnected 0, make pcb ALL CHECKS PASS, sync idempotent, fab outputs
and 3D renders regenerated. 159 parts, still 50 BOM lines, $110.27.

Co-Authored-By: Claude Fable 5.1 <noreply@anthropic.com>
Parts:
- added C50: 4.7uF, Capacitor_SMD:C_0805_2012Metric, symbol Device:C
Connections:
- net GND: now also C50.2
- net VBUS: now also C50.1

Commit message: hardware: BOM from the schematic, JLCPCB fits every part
BOM.csv is now kicad-cli's export of the schematic itself (make pcb-fab),
so every symbol not marked "Exclude from BOM" is on it; gen_jlc reads the
same flags instead of a hand-kept NOT_ASSEMBLED/HAND_SOLDER table.

JLCPCB assembly of the 12 through-hole parts plus LED1 costs ~$22 an order
against ~$110 for partial assembly and a Mouser order, so they are no
longer hand-fitted. Their Assembly field reads "Optional hand solder - JLC
assembles; untick at JLC to fit by hand"; setting it back to "HAND SOLDER"
makes a part hand-fitted again. JLC_PLACEMENT gains fitted corrections for
the six new LCSC parts (J7 needs 180 deg).

LED1 moves to the in-stock WS2812B-V5/W (C2874885): same pinout, and its
VIH of 0.63*VDD (~2.6 V at VLED) is below the old part's 2.7 V.
mouser-order.csv now holds only the mating housings and crimps.

Co-Authored-By: Claude Opus 5.5 <noreply@anthropic.com>
Parts:
- J2: Assembly (none) -> Optional hand solder - JLC assembles; untick at JLC to fit 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
Changed lines of the file:
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@@
 			)
 		)
-	)
+		(property "Assembly" "Optional hand solder - JLC assembles; untick at JLC to fit by hand"
+			(at 77.47 73.66 0)
+			(hide yes)
+			(effects
+				(font
+					(size 1.27 1.27)
+				)
+			)
+		))
 	(symbol
 		(lib_id "Device:C")
