File: hardware/kicad/sheets/ssr.kicad_sch (KiCad schematic)
At the start: 30 parts, among them J4 SSR1, J9 SSR2, Q3 AO3400A, Q4 AO3401A, Q5 CJ2310, Q6 CJ2310, Q7 CJ2310, U10 SN74LVC1G123, U8 TLP291, U9 TLP291

Commit message: hardware: flags at their sources, tri-state MAX31856, Q4 flipped, make erc
Second batch from SCHEMATIC-REVIEW-2026-10-22.md (findings 5, 7, 14, 15,
16 and the local half of 19).

PWR_FLAGs: the power sheet's parked corner is gone. Each flag now sits
where its rail is created - J2.1 (VIN), J2.2 (GND), Q8 source (VIN_P),
L1 output (BUCK_5V) and J1 pin A4 (VBUS, on the mcu sheet) - with the
value text shown on all of them.

MAX31856: U3 and U5 now use bisque:MAX31856 from the new project library
bisque.kicad_sym (registered in sym-lib-table), a copy of the KiCad
symbol with SDO typed tri-state, which is what the part does while CS is
high. The ERC exclusion that papered over the shared SPI_MISO is removed;
ERC is clean with no exclusions.

Q4 is mirrored so the high-side P-FET reads source-up to +5V and drain
down to SSR_EN. One Value string per LCSC part (C38/C44/C45 22uF/25V,
R11 100R 1%); C46 moved 5 mm right to clear the longer text. Every test
point's Value is its net name (TP1 "+3V3" ... TP12 "WDT_CT_P"), so the
board's Value fields, the JLC BOM and the schematic PDF regenerate.

make erc runs kicad-cli ERC at every severity and fails on any
violation; lib_symbol_mismatch, endpoint_off_grid and
same_local_global_label are promoted to errors in the project. It is not
part of pcb-check or CI on purpose.

Board: sync changed only Value fields (0 re-netted); gerbers differ by
timestamp only; DRC 0; full make pcb-check passes.

Co-Authored-By: Claude Fable 5.1 <noreply@anthropic.com>
Parts:
- C38: value 22uF -> 22uF/25V
- TP12: value TP -> WDT_CT_P
Changed lines of the file:
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@@
 	(wire
 		(pts
-			(xy 242.57 92.71) (xy 242.57 90.17)
-		)
-		(stroke
-			(width 0)
-			(type default)
-		)
-	)
-	(wire
-		(pts
 			(xy 227.33 97.79) (xy 234.95 97.79)
 		)
@@
 	(wire
 		(pts
-			(xy 242.57 102.87) (xy 242.57 105.41)
-		)
-		(stroke
-			(width 0)
-			(type default)
-		)
-	)
-	(wire
-		(pts
 			(xy 148.59 110.49) (xy 148.59 100.33)
 		)
@@
 	(wire
 		(pts
-			(xy 242.57 105.41) (xy 246.38 105.41)
+			(xy 177.8 157.48) (xy 177.8 160.02)
 		)
 		(stroke
@@
 	(wire
 		(pts
-			(xy 177.8 157.48) (xy 177.8 160.02)
+			(xy 34.29 168.91) (xy 31.75 168.91)
 		)
 		(stroke
@@
 	(wire
 		(pts
-			(xy 246.38 105.41) (xy 246.38 99.06)
+			(xy 96.52 182.88) (xy 85.09 182.88)
 		)
 		(stroke
@@
 	(wire
 		(pts
-			(xy 34.29 168.91) (xy 31.75 168.91)
+			(xy 242.57 92.71) (xy 242.57 90.17)
 		)
 		(stroke
@@
 	(wire
 		(pts
-			(xy 96.52 182.88) (xy 85.09 182.88)
+			(xy 85.09 82.55) (xy 85.09 92.71)
 		)
 		(stroke
@@
 	(wire
 		(pts
-			(xy 85.09 82.55) (xy 85.09 92.71)
+			(xy 34.29 97.79) (xy 31.75 97.79)
 		)
 		(stroke
@@
 	(wire
 		(pts
-			(xy 34.29 97.79) (xy 31.75 97.79)
+			(xy 62.23 82.55) (xy 59.69 82.55)
 		)
 		(stroke
@@
 	(wire
 		(pts
-			(xy 62.23 82.55) (xy 59.69 82.55)
+			(xy 242.57 102.87) (xy 242.57 105.41)
 		)
 		(stroke
@@
 		)
 	)
+	(label "SSR_EN"
+		(at 242.57 105.41 270)
+		(effects
+			(font
+				(size 1.27 1.27)
+			)
+			(justify right bottom)
+		)
+	)
 	(label "WDT_KICK"
 		(at 191.77 152.4 90)
@@
 	)
 	(label "SSR_EN"
-		(at 242.57 90.17 90)
-		(effects
-			(font
-				(size 1.27 1.27)
-			)
-			(justify left bottom)
-		)
-	)
-	(label "SSR_EN"
 		(at 52.07 92.71 0)
 		(effects
@@
 			)
 		)
-		(property "Value" "22uF"
+		(property "Value" "22uF/25V"
 			(at 171.842 97.47 0)
 			(show_name no)
@@
 			)
 		)
-		(property "Value" "TP"
+		(property "Value" "WDT_CT_P"
 			(at 150.252 101.28 0)
 			(show_name no)
@@
 	)
 	(symbol
-		(lib_id "power:+5V")
-		(at 246.38 99.06 0)
-		(unit 1)
-		(body_style 1)
-		(exclude_from_sim no)
-		(in_bom yes)
-		(on_board yes)
-		(in_pos_files yes)
-		(dnp no)
-		(property "Reference" "#PWR0112"
-			(at 246.38 99.06 0)
-			(hide yes)
-			(show_name no)
-			(do_not_autoplace no)
-			(effects
-				(font
-					(size 1.27 1.27)
-				)
-			)
-		)
-		(property "Value" "+5V"
-			(at 246.38 95.2405 0)
-			(show_name no)
-			(do_not_autoplace no)
-			(effects
-				(font
-					(size 1.27 1.27)
-				)
-			)
-		)
-		(property "Footprint" ""
-			(at 246.38 99.06 0)
-			(hide yes)
-			(show_name no)
-			(do_not_autoplace no)
-			(effects
-				(font
-					(size 1.27 1.27)
-				)
-			)
-		)
-		(property "Datasheet" ""
-			(at 246.38 99.06 0)
-			(hide yes)
-			(show_name no)
-			(do_not_autoplace no)
-			(effects
-				(font
-					(size 1.27 1.27)
-				)
-			)
-		)
-		(property "Description" ""
-			(at 246.38 99.06 0)
-			(show_name no)
-			(do_not_autoplace no)
-			(effects
-				(font
-					(size 1.27 1.27)
-				)
-			)
-		)
-		(pin "1"
-		)
-		(instances
-			(project "bisque-controller"
-				(path "/f24e0cd2-71c5-510c-9d15-562ab64c4388/9f5358df-46db-5b0b-b8f6-c2f90039d70a"
-					(reference "#PWR0112")
-					(unit 1)
-				)
-			)
-		)
-	)
-	(symbol
 		(lib_id "Device:R")
 		(at 22.86 77.47 0)
@@
 	)
 	(symbol
+		(lib_id "power:+5V")
+		(at 242.57 90.17 0)
+		(unit 1)
+		(body_style 1)
+		(exclude_from_sim no)
+		(in_bom yes)
+		(on_board yes)
+		(in_pos_files yes)
+		(dnp no)
+		(property "Reference" "#PWR001"
+			(at 242.57 93.98 0)
+			(hide yes)
+			(show_name no)
+			(do_not_autoplace no)
+			(effects
+				(font
+					(size 1.27 1.27)
+				)
+			)
+		)
+		(property "Value" "+5V"
+			(at 242.57 86.614 0)
+			(show_name no)
+			(do_not_autoplace no)
+			(effects
+				(font
+					(size 1.27 1.27)
+				)
+			)
+		)
+		(property "Footprint" ""
+			(at 242.57 90.17 0)
+			(hide yes)
+			(show_name no)
+			(do_not_autoplace no)
+			(effects
+				(font
+					(size 1.27 1.27)
+				)
+			)
+		)
+		(property "Datasheet" ""
+			(at 242.57 90.17 0)
+			(hide yes)
+			(show_name no)
+			(do_not_autoplace no)
+			(effects
+				(font
+					(size 1.27 1.27)
+				)
+			)
+		)
+		(property "Description" "Power symbol creates a global label with name \"+5V\""
+			(at 242.57 90.17 0)
+			(hide yes)
+			(show_name no)
+			(do_not_autoplace no)
+			(effects
+				(font
+					(size 1.27 1.27)
+				)
+			)
+		)
+		(pin "1"
+		)
+		(instances
+			(project ""
+				(path "/e73561cc-8fa6-5958-924f-c86ad55d4cb9"
+					(reference "#PWR001")
+					(unit 1)
+				)
+			)
+		)
+	)
+	(symbol
 		(lib_id "Isolator:TLP291")
 		(at 41.91 95.25 0)
@@
 		(lib_id "Transistor_FET:AO3401A")
 		(at 240.03 97.79 0)
+		(mirror x)
 		(unit 1)
 		(body_style 1)

Commit message: hardware: honest symbols, real MPNs, U6 spares grounded, LCD_RST verified
Third batch from SCHEMATIC-REVIEW-2026-10-22.md (findings 6, 8, 11, 17,
18 and E1/E2).

Symbols: D8 is bisque:SMAJ30A (drawn as a zener with its cathode on the
rail, since the fitted TVS is unidirectional), Q5-Q7 are bisque:CJ2310
and U2 is bisque:TLV1117LV33, each a flattened copy of the stock symbol
with the fitted part's name, description and LCSC-hosted datasheet, so
no pin or wire moved. The stock D_TVS, 2N7002 and TLV1117-33 embeds are
gone from the sheets.

Sourcing: every one of the 160 assembled symbols now carries MPN (the
manufacturer's part number, from LCSC's product record for its C-number),
Manufacturer and Datasheet (LCSC's hosted PDF) beside LCSC. check_mpn.py
keeps LCSC tied to gen_jlc.LCSC and requires the other two to be present
and MPN not to be a bare C-number.

Drawing: J11's IN1_RAW/IN2_RAW labels read along their own wires instead
of across the connector; U6's unused Darlington inputs I4-I7 are tied to
GND (the board's F.Cu pour already covers them - 4 pads re-netted, 0
unconnected, DRC 0); the root notes record the retired designators and
the LCD_RST finding (the MSP4021's own schematic shows no pull-up on
RESET, so GPIO46 does not block download mode); the mcu sheet notes that
GPIO35/36 rule out R8 (octal PSRAM) modules.

The datasheet manifest maps the shared 22uF/25V sheet to the unified
value and exempts the test points' net-name values. Full make pcb-check
passes; gerbers differ by timestamp and the re-filled GND pour; 3D
renders refreshed.

Co-Authored-By: Claude Fable 5.1 <noreply@anthropic.com>
Parts:
- C38: MPN C12891 -> CL31A226KAHNNNE; Manufacturer (none) -> Samsung Electro-Mechanics
- C39: MPN C49678 -> CC0805KRX7R9BB104; Manufacturer (none) -> YAGEO
- D10, D9: MPN C81598 -> 1N4148W; Manufacturer (none) -> ST(Semtech)
- J4, J9: MPN C8465 -> WJ500V-5.08-2P; Manufacturer (none) -> KANGNEX
- LED3, LED4: MPN C2296 -> KT-0805Y; Manufacturer (none) -> Hubei KENTO Elec
- Q3: MPN C20917 -> AO3400A; Manufacturer (none) -> AOS
- Q4: MPN C15127 -> AO3401A; Manufacturer (none) -> AOS
- Q5, Q6, Q7: symbol Transistor_FET:2N7002 -> bisque:CJ2310; MPN C75882 -> CJ2310; Manufacturer (none) -> JSCJ
- R10, R18, R21: MPN C17414 -> 0805W8F1002T5E; Manufacturer (none) -> UNI-ROYAL
- R19, R6: MPN C17557 -> 0805W8F2200T5E; Manufacturer (none) -> UNI-ROYAL
- R20, R7: MPN C17673 -> 0805W8F4701T5E; Manufacturer (none) -> UNI-ROYAL
- R22, R46, R47, R48, R49: MPN C149504 -> 0805W8F1003T5E; Manufacturer (none) -> UNI-ROYAL
- U10: MPN C123302 -> SN74LVC1G123DCTR; Manufacturer (none) -> TI
- U8, U9: MPN C55144 -> TLP291(GB-TP,SE; Manufacturer (none) -> TOSHIBA

Commit message: hardware: X7R watchdog timing pair, no new feeder (review E5)
R46 100k + C38 22uF X5R 1206 becomes R46 1M (C17514, JLCPCB Basic, the
same UNI-ROYAL 0805 family) with C38 || C49, two 1uF 50V X7R 0805 from
the line C5/C37 already use. The X5R it replaces is unspecified above
85C, loses capacitance to DC bias and ages faster; a single 2.2uF X7R
0805 and every >=10uF 1206 X7R at LCSC are Extended, so two 1uF in
parallel is the fee-free way to an X7R window near the old 2.2 s.

Window 2.0-2.2 s nominal, 1.3-3.1 s worst case with every term a
datasheet or purchase figure - C +-10% tolerance, +-15% over X7R's
whole range, -5% bias and aging, R +-1%, K 1.0-1.1, and the one-shot's
+-0.25uA Rext/Cext leakage, which 1M makes an 11% term (it was 0.8% at
100k; the design note says why that is the price and what would buy it
back). 6.4x margin on the 200 ms kick. The firmware's heartbeat
assertion (900 ms timeout + one kick period inside the minimum window)
moves from 1650 to 1280 ms in tests/host/test_wdt_kick.c, with 180 ms
to spare; make test-host passes. README, Kconfig help, safety.h,
wdt_kick.h, pin-assignments, the firmware backlog and the bench smoke
test carry the new figures.

Board: C49 sits east of C38. To make the room, SSR1_CTRL's F.Cu run
moves to x=61.5 with a jog past LCD_BL's via, and LCD_BL's run moves to
x=62.3 with its via dropped to y=54.5 and two B.Cu segments rejoining
its old path. The two timing nets were ripped up and re-routed by
route.py; U10's WDT_CT_N escape stub is nudged 0.15 mm off C38's pad
corner for check_pcb's rectangular-pad clearance. DRC 0/0 at every
severity, make pcb-check ALL CHECKS PASS, SYNC IDEMPOTENT: PASS; BOM
gains the 1M line and loses nothing, Extended count unchanged at 14.
lcsc_pads.json carries C17514's land pattern; the datasheet manifest
lists the 1M family sheet.

Co-Authored-By: Claude Fable 5.1 <noreply@anthropic.com>
Parts:
- added C49: 1uF, Capacitor_SMD:C_0805_2012Metric, symbol Device:C
- C38: value 22uF/25V -> 1uF; footprint Capacitor_SMD:C_1206_3216Metric -> Capacitor_SMD:C_0805_2012Metric; LCSC C12891 -> C28323; MPN CL31A226KAHNNNE -> CL21B105KBFNNNE
- R46: value 100k -> 1M; LCSC C149504 -> C17514; MPN 0805W8F1003T5E -> 0805W8F1004T5E
Connections:
- net WDT_CT_N: now also C49.1
- net WDT_CT_P: now also C49.2
Changed lines of the file:
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@@
 		)
 	)
+	(wire
+		(pts
+			(xy 168.91 92.71) (xy 179.07 92.71)
+		)
+		(stroke
+			(width 0)
+			(type default)
+		)
+	)
+	(wire
+		(pts
+			(xy 168.91 100.33) (xy 179.07 100.33)
+		)
+		(stroke
+			(width 0)
+			(type default)
+		)
+	)
+	(junction
+		(at 168.91 92.71)
+		(diameter 0)
+		(color 0 0 0 0)
+	)
+	(junction
+		(at 168.91 100.33)
+		(diameter 0)
+		(color 0 0 0 0)
+	)
 	(symbol
 		(lib_id "bisque:CJ2310")
@@
 			)
 		)
-		(property "Value" "22uF/25V"
+		(property "Value" "1uF"
 			(at 171.842 97.47 0)
 			(show_name no)
@@
 			)
 		)
-		(property "Footprint" "Capacitor_SMD:C_1206_3216Metric"
+		(property "Footprint" "Capacitor_SMD:C_0805_2012Metric"
 			(at 168.91 96.52 0)
 			(hide yes)
@@
 			)
 		)
-		(property "Datasheet" "https://datasheet.lcsc.com/datasheet/pdf/02336ea48ea44ca18c72517dd3cb7b47.pdf?productCode=C12891"
+		(property "Datasheet" "https://datasheet.lcsc.com/datasheet/pdf/02336ea48ea44ca18c72517dd3cb7b47.pdf?productCode=C28323"
 			(at 168.91 96.52 0)
 			(hide yes)
@@
 			)
 		)
-		(property "MPN" "CL31A226KAHNNNE"
+		(property "MPN" "CL21B105KBFNNNE"
 			(at 168.91 96.52 0)
 			(hide yes)
@@
 			)
 		)
-		(property "LCSC" "C12891"
+		(property "LCSC" "C28323"
 			(at 168.91 96.52 0)
 			(hide yes)
@@
 	)
 	(symbol
+		(lib_id "Device:C")
+		(at 179.07 96.52 0)
+		(unit 1)
+		(body_style 1)
+		(exclude_from_sim no)
+		(in_bom yes)
+		(on_board yes)
+		(in_pos_files yes)
+		(dnp no)
+		(property "Reference" "C49"
+			(at 182.002 95.57 0)
+			(show_name no)
+			(do_not_autoplace no)
+			(effects
+				(font
+					(size 1.27 1.27)
+				)
+				(justify left)
+			)
+		)
+		(property "Value" "1uF"
+			(at 182.002 97.47 0)
+			(show_name no)
+			(do_not_autoplace no)
+			(effects
+				(font
+					(size 1.27 1.27)
+				)
+				(justify left)
+			)
+		)
+		(property "Footprint" "Capacitor_SMD:C_0805_2012Metric"
+			(at 179.07 96.52 0)
+			(hide yes)
+			(show_name no)
+			(do_not_autoplace no)
+			(effects
+				(font
+					(size 1.27 1.27)
+				)
+			)
+		)
+		(property "Datasheet" "https://datasheet.lcsc.com/datasheet/pdf/02336ea48ea44ca18c72517dd3cb7b47.pdf?productCode=C28323"
+			(at 179.07 96.52 0)
+			(hide yes)
+			(show_name no)
+			(do_not_autoplace no)
+			(effects
+				(font
+					(size 1.27 1.27)
+				)
+			)
+		)
+		(property "Description" "Unpolarized capacitor"
+			(at 179.07 96.52 0)
+			(hide yes)
+			(show_name no)
+			(do_not_autoplace no)
+			(effects
+				(font
+					(size 1.27 1.27)
+				)
+			)
+		)
+		(property "MPN" "CL21B105KBFNNNE"
+			(at 179.07 96.52 0)
+			(hide yes)
+			(show_name no)
+			(do_not_autoplace no)
+			(effects
+				(font
+					(size 1.27 1.27)
+				)
+			)
+		)
+		(property "LCSC" "C28323"
+			(at 179.07 96.52 0)
+			(hide yes)
+			(show_name no)
+			(do_not_autoplace no)
+			(effects
+				(font
+					(size 1.27 1.27)
+				)
+			)
+		)
+		(property "Manufacturer" "Samsung Electro-Mechanics"
+			(at 179.07 96.52 0)
+			(hide yes)
+			(show_name no)
+			(do_not_autoplace no)
+			(effects
+				(font
+					(size 1.27 1.27)
+				)
+			)
+		)
+		(pin "1"
+		)
+		(pin "2"
+		)
+		(instances
+			(project "bisque-controller"
+				(path "/f24e0cd2-71c5-510c-9d15-562ab64c4388/9f5358df-46db-5b0b-b8f6-c2f90039d70a"
+					(reference "C49")
+					(unit 1)
+				)
+			)
+		)
+	)
+	(symbol
 		(lib_id "Device:R")
 		(at 22.86 148.59 0)
@@
 			)
 		)
-		(property "Value" "100k"
+		(property "Value" "1M"
 			(at 160.666 97.47 0)
 			(show_name no)
@@
 			)
 		)
-		(property "Datasheet" "https://datasheet.lcsc.com/datasheet/pdf/0a975aaa49b7c97f38a963127be4a823.pdf?productCode=C149504"
+		(property "Datasheet" "https://datasheet.lcsc.com/datasheet/pdf/0a975aaa49b7c97f38a963127be4a823.pdf?productCode=C17514"
 			(at 158.75 96.52 0)
 			(hide yes)
@@
 			)
 		)
-		(property "MPN" "0805W8F1003T5E"
+		(property "MPN" "0805W8F1004T5E"
 			(at 158.75 96.52 0)
 			(hide yes)
@@
 			)
 		)
-		(property "LCSC" "C149504"
+		(property "LCSC" "C17514"
 			(at 158.75 96.52 0)
 			(hide yes)

Commit message: hardware: the five quick fixes from the 2026-10-05/10-22 reviews
Schematic (rev B.3, sheets ct/power/mcu/ssr + root):
- R65, 1k from CTA_P to GND, mirrors R33 so the floating CT secondary
  sits at +-V/2 on IAP/IAN and channel A's pin limit is 139 A nominal,
  the same as channel B (schematic review 10-05 item 2).
- D9/D10 freewheel diodes are B5819W (JSCJ C8598, Basic, 1 A / 40 V,
  9 A surge) in the same SOD-123 land, replacing the 1N4148W whose
  150 mA rating never covered a 200 mA contactor coil (PCB review 10-05
  item 12). The SS34 was tried first and does not fit the SSR column.
- ADE_RESET is a hierarchical net to U1 IO37, the spare GPIO; the R30/C37
  RC stays for the power-on stretch (10-22 review E3).
- PWR_STATUS: BUCK_5V through R66 (100k) over R67+R68 (130k) to U1 IO45,
  2.8 V when the 24 V buck runs and 0 V on USB only (10-22 review E4).
  The TPS2116 ST pin would have said the same thing but its pad is boxed
  in by the USB pair on this layout, so it stays unconnected (C3, rev C).

Board:
- Every +5V layer transition (7) now has a second 0.6/0.3 via 0.85 mm
  away with a stub on each layer; the two in the USB corner use 0.3 mm
  stubs (fab-readiness C, "attempted, not landed" -> fixed).
- R65 placed below the CT filters; the divider in the two free columns
  south of U1, lifted 0.75 mm so the nameplate pocket keeps its 16.2 mm
  (it prints at 62% now). BUCK_5V tap hand-routed, the rest by the
  in-house router. DRC 0, make pcb-check ALL CHECKS PASS, 3D re-rendered.

Firmware/docs: KILN_PIN_ADE_RESET (37) and KILN_PIN_PWR_STATUS (45) in
Kconfig with the GPIO45 strapping caveat, check_pinmap NET_KCONFIG,
docs/pin-assignments.md (all 30 GPIOs assigned), DESIGN-NOTES sections
for each change, status notes in the four review documents, gen_jlc
sourcing + JLC_PLACEMENT rows, lcsc_pads cache and datasheet manifest.

Co-Authored-By: Claude Fable 5.1 <noreply@anthropic.com>
Parts:
- D10, D9: value 1N4148W -> B5819W; symbol Device:D -> Device:D_Schottky; LCSC C81598 -> C8598; MPN 1N4148W -> B5819W SL; Manufacturer ST(Semtech) -> JSCJ
Changed lines of the file:
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@@
 	)
 	(symbol
-		(lib_id "Device:D")
+		(lib_id "Device:D_Schottky")
 		(at 66.04 153.67 0)
 		(unit 1)
@@
 			)
 		)
-		(property "Value" "1N4148W"
+		(property "Value" "B5819W"
 			(at 62.23 150.49 0)
 			(show_name no)
@@
 			)
 		)
-		(property "Datasheet" "https://datasheet.lcsc.com/datasheet/pdf/8abd7fc00ebe41ffb03ad1383c10753b.pdf?productCode=C81598"
+		(property "Datasheet" "https://datasheet.lcsc.com/datasheet/pdf/4ac2c059be7c462694ab0715ce987a85.pdf?productCode=C8598"
 			(at 66.04 153.67 0)
 			(hide yes)
@@
 			)
 		)
-		(property "Description" "Diode"
+		(property "Description" "Schottky diode"
 			(at 66.04 153.67 0)
 			(hide yes)
@@
 			)
 		)
-		(property "MPN" "1N4148W"
+		(property "MPN" "B5819W SL"
 			(at 66.04 153.67 0)
 			(hide yes)
@@
 			)
 		)
-		(property "LCSC" "C81598"
+		(property "LCSC" "C8598"
 			(at 66.04 153.67 0)
 			(hide yes)
@@
 			)
 		)
-		(property "Manufacturer" "ST(Semtech)"
+		(property "Manufacturer" "JSCJ"
 			(at 66.04 153.67 0)
 			(hide yes)
@@
 	)
 	(symbol
-		(lib_id "Device:D")
+		(lib_id "Device:D_Schottky")
 		(at 66.04 82.55 0)
 		(unit 1)
@@
 			)
 		)
-		(property "Value" "1N4148W"
+		(property "Value" "B5819W"
 			(at 62.23 79.37 0)
 			(show_name no)
@@
 			)
 		)
-		(property "Datasheet" "https://datasheet.lcsc.com/datasheet/pdf/8abd7fc00ebe41ffb03ad1383c10753b.pdf?productCode=C81598"
+		(property "Datasheet" "https://datasheet.lcsc.com/datasheet/pdf/4ac2c059be7c462694ab0715ce987a85.pdf?productCode=C8598"
 			(at 66.04 82.55 0)
 			(hide yes)
@@
 			)
 		)
-		(property "Description" "Diode"
+		(property "Description" "Schottky diode"
 			(at 66.04 82.55 0)
 			(hide yes)
@@
 			)
 		)
-		(property "MPN" "1N4148W"
+		(property "MPN" "B5819W SL"
 			(at 66.04 82.55 0)
 			(hide yes)
@@
 			)
 		)
-		(property "LCSC" "C81598"
+		(property "LCSC" "C8598"
 			(at 66.04 82.55 0)
 			(hide yes)
@@
 			)
 		)
-		(property "Manufacturer" "ST(Semtech)"
+		(property "Manufacturer" "JSCJ"
 			(at 66.04 82.55 0)
 			(hide yes)
