File: hardware/kicad/sheets/test.kicad_sch (KiCad schematic)
At the start: 18 parts

Commit message: hardware: hierarchical schematic, ERC at 0/0, rev B.3
Applies items 1-3 of SCHEMATIC-REVIEW-2026-10-22.md.

ERC: the 173 lib_symbol_mismatch warnings were over-escaped quotes in the
embedded power symbols' Description strings; refreshed from the library.
The 18 off-grid power symbols are snapped and their stub wires redrawn.
The VIN and VLED global labels that existed only to carry a PWR_FLAG are
gone; the flags now sit on the nets they drive (J2.1, the VLED junction).
ERC reads 0 errors / 0 warnings with the documented SDO exclusion.

Hierarchy: no global labels remain. Each net that crosses sheets has one
hierarchical label per sheet, matching sheet pins on the root, and the
root wires those pins as a block diagram. Every other former global label
is a local label. The eight signal test points (TP4-TP11) move from the
test sheet to the mcu and ct sheets beside their nets, so the test block
needs no pins. KiCad names the nets /mcu/SPI_MISO etc.; netlist.py strips
the path, so the board's net names and the routing tables are unchanged
(182 components, 538 pads, 0 mismatches). single_global_label is now a
warning. check_sync_idempotent's collision fixture used the bare
"SPI_MISO" name and is updated, with a loud failure if its victims vanish.

Drawing: rev B.3 dated 2026-10-22 on every sheet, ct on A3 like the rest,
the three overflowing titles shortened, and the notes no longer refer to
design.py or to crystal load caps that no longer exist.

Co-Authored-By: Claude Fable 5.1 <noreply@anthropic.com>
Parts:
- removed TP10, TP11, TP4, TP5, TP6, TP7, TP8, TP9: TP, TestPoint:TestPoint_Pad_D1.0mm, symbol Connector:TestPoint
Other:
- note added: "MOUNTING / FIDUCIALS FID1-3 are bare-copper pick-and-place targets, on no net"
- note removed: "MOUNTING / FIDUCIALS / POWER FLAGS FID1-3 are bare-copper pick-and-place targets, on no net"
- title: Bisque Kiln Controller - Test points, mounting, fiducials, power flags -> Bisque Kiln Controller - Test points and mounting

Commit message: hardware: flags at their sources, tri-state MAX31856, Q4 flipped, make erc
Second batch from SCHEMATIC-REVIEW-2026-10-22.md (findings 5, 7, 14, 15,
16 and the local half of 19).

PWR_FLAGs: the power sheet's parked corner is gone. Each flag now sits
where its rail is created - J2.1 (VIN), J2.2 (GND), Q8 source (VIN_P),
L1 output (BUCK_5V) and J1 pin A4 (VBUS, on the mcu sheet) - with the
value text shown on all of them.

MAX31856: U3 and U5 now use bisque:MAX31856 from the new project library
bisque.kicad_sym (registered in sym-lib-table), a copy of the KiCad
symbol with SDO typed tri-state, which is what the part does while CS is
high. The ERC exclusion that papered over the shared SPI_MISO is removed;
ERC is clean with no exclusions.

Q4 is mirrored so the high-side P-FET reads source-up to +5V and drain
down to SSR_EN. One Value string per LCSC part (C38/C44/C45 22uF/25V,
R11 100R 1%); C46 moved 5 mm right to clear the longer text. Every test
point's Value is its net name (TP1 "+3V3" ... TP12 "WDT_CT_P"), so the
board's Value fields, the JLC BOM and the schematic PDF regenerate.

make erc runs kicad-cli ERC at every severity and fails on any
violation; lib_symbol_mismatch, endpoint_off_grid and
same_local_global_label are promoted to errors in the project. It is not
part of pcb-check or CI on purpose.

Board: sync changed only Value fields (0 re-netted); gerbers differ by
timestamp only; DRC 0; full make pcb-check passes.

Co-Authored-By: Claude Fable 5.1 <noreply@anthropic.com>
Parts:
- TP1: value TP -> +3V3
- TP2: value TP -> +5V
- TP3: value TP -> GND
Changed lines of the file:
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@@
 			)
 		)
-		(property "Value" "TP"
+		(property "Value" "GND"
 			(at 47.382 37.78 0)
 			(show_name no)
@@
 			)
 		)
-		(property "Value" "TP"
+		(property "Value" "+3V3"
 			(at 24.522 42.86 0)
 			(show_name no)
@@
 			)
 		)
-		(property "Value" "TP"
+		(property "Value" "+5V"
 			(at 35.952 42.86 0)
 			(show_name no)

Commit message: hardware: drop the five test points a connector already exposes
TP1 (+3V3), TP2 (+5V), TP7/TP8 (I2C) and TP11 (CTA_P) each sat on a net
that a connector pin already reaches: +3V3 and I2C on the J7 AUX header
and J14 QWIIC, +5V on J5 pin 1, CTA_P on J12 pin 1. They are gone from
the test, mcu and ct sheets (TP3 and TP9/TP10 slide left into the gaps),
the board is synced, and the copper that only existed to reach them is
removed: eight segments and one via, 15.5 mm in all, most of it +5V's
spur from U2.3 up to the old TP2. DRC is 0 violations / 0 unconnected
with every severity on.

The seven that remain (TP3-TP6, TP9, TP10, TP12) probe nets nothing else
reaches, and none moved: on the board each already sits inline on its
net's route with at most a 0.4 mm jog. TP12 is the one with a real stub
(3.3 mm from R46.2), and SJ2's courtyard is what keeps it there.

TP_LEGEND_OK is empty again - dropping TP11 was the way out review A2
named. README, the bench smoke test (rails now probed at C2 / J7 pin 1),
gen_jlc's not-assembled set and the datasheet manifest follow. ERC 0,
make pcb-check ALL CHECKS PASS, SYNC IDEMPOTENT: PASS; fab outputs and
3D renders regenerated.

Co-Authored-By: Claude Fable 5.1 <noreply@anthropic.com>
Parts:
- removed TP1: +3V3, TestPoint:TestPoint_Pad_D1.0mm, symbol Connector:TestPoint
- removed TP2: +5V, TestPoint:TestPoint_Pad_D1.0mm, symbol Connector:TestPoint
Other:
- moved on the sheet: TP3

Commit message: hardware: BOM from the schematic, JLCPCB fits every part
BOM.csv is now kicad-cli's export of the schematic itself (make pcb-fab),
so every symbol not marked "Exclude from BOM" is on it; gen_jlc reads the
same flags instead of a hand-kept NOT_ASSEMBLED/HAND_SOLDER table.

JLCPCB assembly of the 12 through-hole parts plus LED1 costs ~$22 an order
against ~$110 for partial assembly and a Mouser order, so they are no
longer hand-fitted. Their Assembly field reads "Optional hand solder - JLC
assembles; untick at JLC to fit by hand"; setting it back to "HAND SOLDER"
makes a part hand-fitted again. JLC_PLACEMENT gains fitted corrections for
the six new LCSC parts (J7 needs 180 deg).

LED1 moves to the in-stock WS2812B-V5/W (C2874885): same pinout, and its
VIH of 0.63*VDD (~2.6 V at VLED) is below the old part's 2.7 V.
mouser-order.csv now holds only the mating housings and crimps.

Co-Authored-By: Claude Opus 5.5 <noreply@anthropic.com>
Parts:
- FID1, FID2, FID3, H1, H2, H3, H4, TP3: now left out of the parts list
Changed lines of the file:
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@@
 		(body_style 1)
 		(exclude_from_sim no)
-		(in_bom yes)
+		(in_bom no)
 		(on_board yes)
 		(in_pos_files yes)
@@
 		(body_style 1)
 		(exclude_from_sim no)
-		(in_bom yes)
+		(in_bom no)
 		(on_board yes)
 		(in_pos_files yes)
@@
 		(body_style 1)
 		(exclude_from_sim no)
-		(in_bom yes)
+		(in_bom no)
 		(on_board yes)
 		(in_pos_files yes)
@@
 		(body_style 1)
 		(exclude_from_sim no)
-		(in_bom yes)
+		(in_bom no)
 		(on_board yes)
 		(in_pos_files yes)
@@
 		(body_style 1)
 		(exclude_from_sim no)
-		(in_bom yes)
+		(in_bom no)
 		(on_board yes)
 		(in_pos_files yes)
@@
 		(body_style 1)
 		(exclude_from_sim no)
-		(in_bom yes)
+		(in_bom no)
 		(on_board yes)
 		(in_pos_files yes)
@@
 		(body_style 1)
 		(exclude_from_sim no)
-		(in_bom yes)
+		(in_bom no)
 		(on_board yes)
 		(in_pos_files yes)
@@
 		(body_style 1)
 		(exclude_from_sim no)
-		(in_bom yes)
-		(on_board yes)
-		(in_pos_files yes)
+		(in_bom no)
+		(on_board yes)
+		(in_pos_files yes)
